File: kicad/YAWC/YAWC.kicad_sch (KiCad schematic)
At the start: 143 parts, among them J1 Screw_Terminal_01x04, J10 Screw_Terminal_01x03, J11 Screw_Terminal_01x03, J12 PSU_OUT, J13 Conn_01x03, J2 Screw_Terminal_01x04, J3 Screw_Terminal_01x04, J4 Screw_Terminal_01x04, J5 Input, J6 PSU_IN, J7 SSR, J8 Screw_Terminal_01x03, J9 Screw_Terminal_01x03, Q1 NMOS, Q10 NMOS, Q11 NMOS, Q12 NMOS, Q13 BSS138, Q2 NMOS, Q3 NMOS, Q4 NMOS, Q5 NMOS, Q6 NMOS, Q7 NMOS, Q8 NMOS, Q9 NMOS, U1 LCKFB-ESP32S3R8N8, U10 BME280, U11 TSOP382xx, U2 TC4427xOA, U3 TC4427xOA, U4 TC4427xOA, U5 TC4427xOA, U6 TC4427xOA, U7 TC4427xOA, U8 K7805-1000R3, U9 74AHCT125

Commit message: parts assign
finished part assignement.
Parts:
- C1, C11, C3, C33, C34, C5, C7, C9: LCSC (none) -> C1591
- C10, C12, C13, C14, C17, C18, C19, C2, C20, C21, C22, C23, C24, C35, C4, C6, C8: LCSC (none) -> C138687
- D1, D2, D3, D4, D5, D6, D7, D8: LCSC (none) -> C224017
- F10: LCSC (none) -> C19727305
- F5: LCSC (none) -> C108518
- J1, J12, J2, J3, J4, J7: footprint (none) -> TerminalBlock:TerminalBlock_bornier-4_P5.08mm; LCSC (none) -> C2915641
- J10, J11, J5, J6, J8, J9: footprint (none) -> TerminalBlock:TerminalBlock_bornier-3_P5.08mm; LCSC (none) -> C72334
- J13: footprint (none) -> Connector_PinHeader_2.54mm:PinHeader_1x03_P2.54mm_Vertical
- Q1, Q10, Q11, Q12, Q2, Q3, Q4, Q5, Q6, Q7, Q8, Q9: footprint (none) -> Package_TO_SOT_SMD:Infineon_PG-HSOF-8-1; LCSC (none) -> C42403238
- Q13: LCSC (none) -> C52895
- R1, R10, R11, R12, R2, R3, R4, R5, R6, R7, R8, R9: value R -> 12r; footprint (none) -> Resistor_SMD:R_0603_1608Metric; LCSC (none) -> C246021
- R13, R14, R15, R16, R17, R18, R19, R20, R21, R22, R23, R24, R25, R27, R28, R29, R30, R31, R32, R33, R34, R35, R36, R37, R38, R39: footprint (none) -> Resistor_SMD:R_0603_1608Metric; LCSC (none) -> C15401
- R26: LCSC (none) -> C2933801
- RV1: footprint (none) -> Varistor:RV_Disc_D12mm_W5.4mm_P7.5mm
- U10: LCSC (none) -> C92489
- U11: LCSC (none) -> C141632
- U2, U3, U4, U5, U6, U7: LCSC (none) -> C20551
- U9: LCSC (none) -> C554502
Connections:
- net ARGB_1: now also U9.3; no longer U9.11
- net ARGB_2: no longer U9.8
- net ARGB_3: no longer U9.6
- net ARGB_4: now also U9.11; no longer U9.3
- net at R30.2: now also Q11.2 (G), R11.1
Other:
- note added: "ext switch"
- moved on the sheet: R30

Commit message: finished pcb routing
basically finished i suppose ?
Parts:
- removed C10, C12, C13, C8: 10u, Capacitor_SMD:C_1210_3225Metric, symbol Device:C
- removed C11, C9: 100n, Capacitor_SMD:C_0603_1608Metric, symbol Device:C
- removed C27, C28, C29, C30, C31, C32: 470u, Capacitor_THT:CP_Radial_D10.0mm_P5.00mm, symbol Device:C_Polarized
- added R40: 10k, Resistor_SMD:R_0603_1608Metric, symbol Device:R
- C15: value 100n -> 10n; footprint Capacitor_THT:C_Rect_L26.5mm_W8.5mm_P22.50mm_MKS4 -> Capacitor_THT:C_Rect_L13.0mm_W4.0mm_P10.00mm_FKS3_FKP3_MKS4; LCSC C3295436 -> C428926
- F1, F10, F2, F3, F4, F6, F7, F8, F9: footprint easyeda2kicad:FUSE-TH_4P-L16.0-W6.7 -> lib:FUSE-TH_4P-L16.0-W6.7
- Q1, Q10, Q11, Q12, Q2, Q3, Q4, Q5, Q6, Q7, Q8, Q9: footprint Package_TO_SOT_SMD:Infineon_PG-HSOF-8-1 -> lib:Infineon_PG-HSOF-8-1
- U1: footprint easyeda2kicad:DIP-40_L20.32-W51.66-P2.54-LS15.24 -> lib:DIP-40_L20.32-W51.66-P2.54-LS15.24
Connections:
- net +24V: no longer D10.1 (A1), D11.1 (A1), D12.1 (A1), D13.1 (A1), D14.1 (A1), D15.1 (A1), D16.1 (A1), D17.1 (A1), D18.1 (A1), D19.1 (A1), D20.1 (A1), D9.1 (A1)
- net ARGB_1: now also U9.11; no longer U9.3
- net ARGB_2: now also U9.8
- net ARGB_3: now also U9.3
- net ARGB_4: now also U9.6; no longer U9.11
- net GND: now also R40.1
- net LINE: now also J7.1 (Pin_1); no longer J7.2 (Pin_2)
- net B24: now reaches F2.1, J2.4 (Pin_4)
- net B24: now also D12.1 (A1), D13.1 (A1), D14.1 (A1)
- net A24: now reaches F1.1, J1.4 (Pin_4)
- net A24: now also D10.1 (A1), D11.1 (A1), D9.1 (A1)
- net D24: now reaches F4.1, J4.4 (Pin_4)
- net D24: now also D18.1 (A1), D19.1 (A1), D20.1 (A1)
- net at U1.35 (G16): now also U9.2; no longer U9.5
- net at U1.36 (G15): now also U9.5; no longer U9.2
- net C24: now reaches F3.1, J3.4 (Pin_4)
- net C24: now also D15.1 (A1), D16.1 (A1), D17.1 (A1)
- net at Q8.2 (G), R8.1: now also R40.2
- net at R29.2: now also Q12.2 (G), R12.1
- net at J6.1 (Pin_1): now also J7.2 (Pin_2); no longer J7.1 (Pin_1)
Other:
- moved on the sheet: C7, R29, U9A, U9B
